File: gamepad_electronics/gamepad_electronics.kicad_pcb (KiCad board)
At the start: 2 copper layers, 100 x 50 mm, 97 parts, among them J1 USB_C_Receptacle_USB2.0_16P, M1 VIBRATOR_1, M2 VIBRATOR_2, Q1 AO3400A, Q2 AO3400A, Q3 FS8205A, Q4 AO3401A, Q5 AO3401A, SW1 DPAD_UP, SW2 DPAD_RIGHT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

Commit message: fix
Parts:
- U4: footprint tp4056:SOP127P600X175-9N -> Package_SO:HTSOP-8-1EP_3.9x4.9mm_P1.27mm_EP2.4x3.2mm_ThermalVias
Other:
- outline, holes or cut-outs redrawn
