File: gamepad_electronics/supply.kicad_sch (KiCad schematic)
At the start: 35 parts, among them Q3 FS8205A, Q4 AO3401A, Q5 AO3401A, SW9 PWR_SW, U4 TP4056, U5 MT3608, U6 AMS1117-3.3, U7 DW01A

Commit message: fix
Parts:
- U4: footprint tp4056:SOP127P600X175-9N -> Package_SO:HTSOP-8-1EP_3.9x4.9mm_P1.27mm_EP2.4x3.2mm_ThermalVias
Changed lines of the file:
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@@
 			)
 		)
-		(property "Footprint" "tp4056:SOP127P600X175-9N"
+		(property "Footprint" "Package_SO:HTSOP-8-1EP_3.9x4.9mm_P1.27mm_EP2.4x3.2mm_ThermalVias"
 			(at 69.596 26.416 0)
 			(effects
